File: pcb/POTENCIOSTATO_22-11-2018.brd (EAGLE design)
At the start: 56 x 64.9 mm, 45 parts, among them IC1 TL074P, IC2 TL074P, K2 ZNS5406, Q1 2N3904

Commit message: Atualização da pcb. Versão final
Routing:
- net GND: track 242.0 -> 229.8 mm
- net 5V: track 135.8 -> 133.4 mm
- net N$10: track 23.3 -> 24.5 mm
- net N$18: track 50.1 -> 49.4 mm
- net N$13: track 6.15 -> 6.76 mm
- net WEL: track 132.7 -> 132.2 mm
