File: pcb/pcb_homemade/potenciostato_last.sch (EAGLE design)
At the start: 34 parts, among them IC1 LM741P, IC2 TL074P, K2 ZNS5406, Q1 2N3904

Commit message: Final_version, imprimir layout para confirmar
Parts:
- removed IC1: LM741P, linear:LM741P
- removed IC2: TL074P, linear:TL074P
- removed JP6, JP7: (no value), pinhead:PINHD-1X1
- removed LED2: TLLG4400, led:TLLG4400
- removed R15: 1K, rcl:R-EU_0207/7
- added C6, C7, C8: 1uF, rcl:C-EU050-035X075
- added IC3: TL074P, linear:TL074P
Connections:
- removed net N$13: R8.1, SW1.4
- net 3V3: now also IC3P.V+; no longer IC1.V+, IC2P.V+
- net 5V: no longer R15.1
- net AD: now also IC3B.OUT, SW1.6; no longer C4.2, IC2D.OUT
- net AUX: now also IC3D.OUT; no longer IC2C.OUT
- net DA: now also R4.2; no longer IC2A.+IN
- net GND: now also IC3P.V-; no longer IC1.V-, IC2P.V-, JP1.25, JP3.1, JP6.1, JP7.1, LED2.C
- net N$1: now also C4.2, R8.1, SW1.4; no longer IC2A.-IN, IC2A.OUT, R4.2
- net N$10: now also C6.2
- net N$11: now also C7.2
- net N$12: now also C8.2
- net N$2: now also IC3C.-IN, IC3C.OUT; no longer IC2B.-IN, IC2B.OUT
- net N$3: now also IC3A.+IN; no longer IC1.+IN
- net N$4: now also IC3D.-IN; no longer IC2C.-IN
- net N$6: now also IC3D.+IN; no longer IC2C.+IN
- net N$7: now also JP3.1; no longer LED2.A, R15.2
- net N$8: now also IC3B.+IN; no longer IC2D.+IN
- net REFEL: now also IC3C.+IN; no longer IC2B.+IN
- net VCC/2: now also IC3A.-IN, IC3A.OUT; no longer IC1.-IN, IC1.OUT
- net WEL: now also C6.1, C7.1, C8.1, IC3B.-IN, SW1.7; no longer IC2D.-IN
Other:
- moved on the sheet: R10, R11, R8, SW1
