File: pcb/pcb_pro/potenciostato_last.sch (EAGLE design)
At the start: 25 parts, among them IC1 LM741P, IC2 TL074P, K2 ZNS5406, Q1 2N3904

Commit message: Final_version, imprimir layout para confirmar
Parts:
- removed IC1: LM741P, linear:LM741P
- removed IC2: TL074P, linear:TL074P
- removed R12: 47, rcl:R-EU_0207/7
- added C6, C7, C8: 1uF, rcl:C-EU050-035X075
- added IC3: TL074P, linear:TL074P
- added JP1: (no value), pinhead:PINHD-2X20/90
- added JP2, JP3, JP4, JP5: (no value), pinhead:PINHD-1X1
- added X1: (no value), con-ptr500:AK500/4
Connections:
- removed net N$13: R8.1, SW1.5
- new net N$7: JP3.1
- net 3V3: now also IC3P.V+, JP1.1; no longer IC1.V+, IC2P.V+
- net 5V: now also JP1.2
- net AD: now also IC3B.OUT, JP4.1, SW1.5, SW1.6; no longer C4.2, IC2D.OUT, SW1.10, SW1.11, SW1.12, SW1.8, SW1.9
- net AUX: now also IC3D.OUT; no longer IC2C.OUT
- net AUXEL: now also X1-2.KL
- net DA: now also JP2.1, R4.2; no longer IC2A.+IN
- net GND: now also IC3P.V-, JP1.39, JP5.1, X1-1.KL; no longer IC1.V-, IC2P.V-
- net GPIO: now also JP1.29
- net N$1: now also C4.2, R8.1, SW1.4; no longer IC2A.-IN, IC2A.OUT, R4.2
- net N$10: now also C6.2, SW1.1; no longer SW1.2
- net N$11: now also C7.2, SW1.2; no longer SW1.3
- net N$12: now also C8.2, SW1.3; no longer SW1.4
- net N$2: now also IC3C.-IN, IC3C.OUT; no longer IC2B.-IN, IC2B.OUT
- net N$3: now also IC3A.+IN; no longer IC1.+IN
- net N$4: now also IC3D.-IN; no longer IC2C.-IN
- net N$6: now also IC3D.+IN; no longer IC2C.+IN
- net N$8: now also IC3B.+IN; no longer IC2D.+IN
- net N$9: now also SW1.10, SW1.11, SW1.12, SW1.8, SW1.9; no longer R12.1, SW1.1
- net REFEL: now also IC3C.+IN, X1-3.KL; no longer IC2B.+IN
- net VCC/2: now also IC3A.-IN, IC3A.OUT; no longer IC1.-IN, IC1.OUT
- net WEL: now also C6.1, C7.1, C8.1, IC3B.-IN, SW1.7, X1-4.KL; no longer IC2D.-IN, R12.2
Other:
- moved on the sheet: R10, R11, R8, SW1
