File: pcb/pcb_pro/potenciostato_last.brd (EAGLE design)
At the start: 65.3 x 56.6 mm, 32 parts, among them IC3 TL074P, K2 ZNS5406, Q1 2N3904

Commit message: Final_version, imprimir layout para confirmar WIP
Parts:
- moved SW1 3.38 mm to (5.95, 57.3)
- moved X1 3.23 mm to (3.52, 77.8)
- moved C2 2.38 mm to (57.2, 49.7)
- moved C3 0.91 mm to (57.0, 61.1)
- moved R3 0.40 mm to (57.5, 66.4)
- moved JP1 0.14 mm to (31.6, 99.0)
Routing:
- net GND: track 270.2 -> 173.2 mm, vias 0 -> 8
- net REFEL: track 119.9 -> 38.3 mm, vias 0 -> 1
- net WEL: track 95.9 -> 100.8 mm
- net N$1: track 12.6 -> 16.2 mm
- net N$12: track 22.6 -> 25.7 mm
- net N$11: track 31.6 -> 34.7 mm
- net AUXEL: track 45.0 -> 47.5 mm
- net 3V3: track 173.1 -> 175.4 mm
- net AD: track 56.6 -> 54.5 mm
- net N$10: track 41.5 -> 43.4 mm
- net 5V: track 105.2 -> 103.6 mm
- added copper zone on layer 1, net GND
